Commit message: Add robust training setup with crash recovery
- Increase checkpoint frequency from 50k to 10k steps (reduces max loss from 10% to 2%)
- Add comprehensive error handling with emergency model save on exceptions
- Add curriculum state persistence to JSON every 100 episodes
- Initialize last_distance/last_alignment attributes to prevent AttributeError
- Fix hardcoded paths from /home/iqraq/ to /home/Master/ in all files
- Fix malformed float literal 00.1 to 0.1 in C1.py
- Add shimmy dependency for gym compatibility

Co-Authored-By: Claude Opus 4.5 <noreply@anthropic.com>

File: Cube.urdf (robot description, URDF)
Before this commit: robot stl_object, 1 links, 0 joints
Links:
- link base_link: geometry collision mesh filename=/home/Master/Cube.stl scale=1 1 1; visual mesh filename=/home/Master/Cube.stl scale=1 1 1

File: Inspection_Station.urdf (robot description, URDF)
Before this commit: robot stl_object, 1 links, 0 joints
Links:
- link base_link: geometry visual mesh filename=/home/Master/Inspection_Station.stl scale=1 1 1

File: mycobot_urdf_copy.urdf (robot description, URDF)
Before this commit: robot firefighter, 9 links, 8 joints
Links:
- link joint1: geometry collision mesh filename=/home/Master/meshes/joint1.dae; visual mesh filename=/home/Master/meshes/joint1.dae
- link joint2: geometry collision mesh filename=/home/Master/meshes/joint2.dae; visual mesh filename=/home/Master/meshes/joint2.dae
- link joint3: geometry collision mesh filename=/home/Master/meshes/joint3.dae; visual mesh filename=/home/Master/meshes/joint3.dae
- link joint4: geometry collision mesh filename=/home/Master/meshes/joint4.dae; visual mesh filename=/home/Master/meshes/joint4.dae
- link joint5: geometry collision mesh filename=/home/Master/meshes/joint5.dae; visual mesh filename=/home/Master/meshes/joint5.dae
- link joint6: geometry collision mesh filename=/home/Master/meshes/joint6.dae; visual mesh filename=/home/Master/meshes/joint6.dae
- link joint6_flange: geometry collision mesh filename=/home/Master/meshes/joint7.dae; visual mesh filename=/home/Master/meshes/joint7.dae
